File: teensynth.kicad_pcb (KiCad board)
At the start: 2 copper layers, 89 parts, among them CON1 SJ-3523-SMT-TR, CON2 SJ-3523-SMT-TR, J1 Control_0, J10 LED_3_O, J11 LED_3_I, J12 LED_0_I, J13 LED_2_O, J14 Control_2, J15 Control_6, J16 LED_2_I, J17 LED_X_O, J18 LED_1_O, J19 LED_X_I, J2 Control_4, J20 Control_3, J21 Control_7, J22 LED_1_I, J23 LED_0_O, J24 10118193-0001LF, J25 10118193-0001LF, J3 LED_4_O, J4 LED_5_0, J5 LED_5_I, J6 LED_4_I, J7 Control_1, J8 Control_5, J9 LED_6_I, U1 CD74HC4051E, U2 MCP23017-E_SP, U3 Teensy3.2

Commit message: Throw everything in a reasonable place
Parts:
- U1: footprint digikey-footprints:DIP-16_W7.62mm -> digikey-footprints:SOIC-16_W7.5mm
- U2: footprint digikey-footprints:DIP-28_W7.62mm -> digikey-footprints:SOIC-28_W7.5mm
- moved R8 328.8 mm to (326.4, 139.7)
- moved CON1 323.8 mm to (330.0, 68.6), turned to 180 degrees
- moved CON2 287.6 mm to (306.4, 68.6)
- moved J19 256.7 mm to (283.2, 83.8), turned to 180 degrees
- moved J12 251.6 mm to (334.0, 55.9), turned to 270 degrees
- moved J17 250.4 mm to (273.1, 83.8), turned to 180 degrees
- moved R1 250.4 mm to (266.7, 62.2), turned to 90 degrees
- moved D10 249.2 mm to (288.3, 81.3), turned to 90 degrees
- moved J21 247.7 mm to (328.9, 143.5)
- moved R3 184.0 mm to (204.5, 62.2), turned to 90 degrees
- moved J4 163.3 mm to (34.3, 147.3), turned to 180 degrees
- moved J1 160.1 mm to (270.5, 61.0), turned to 90 degrees
- moved J23 148.7 mm to (278.1, 69.8), turned to 90 degrees
- moved J22 148.3 mm to (271.8, 66.0), turned to 270 degrees
- moved R4 143.6 mm to (25.4, 151.1), turned to 180 degrees
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
Commit message: Update design rules
Other:
- net class Default: trace_width 0.25 -> 0.2; via_dia 0.8 -> 0.6; via_drill 0.4 -> 0.3
- net class Power added: clearance 0.2, trace_width 0.7, via_dia 1, via_drill 0.5
- net class Test removed
- rule via_min_size: 0.4 -> 0.6
Changed lines of the file:
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@@
   )
   (setup
-    (last_trace_width 0.25)
+    (last_trace_width 0.2)
     (trace_clearance 0.2)
     (zone_clearance 0.508)
@@
     (segment_width 0.2)
     (edge_width 0.1)
-    (via_size 0.8)
-    (via_drill 0.4)
-    (via_min_size 0.4)
+    (via_size 0.6)
+    (via_drill 0.3)
+    (via_min_size 0.6)
     (via_min_drill 0.3)
-    (uvia_size 0.3)
-    (uvia_drill 0.1)
+    (uvia_size 0.6)
+    (uvia_drill 0.3)
     (uvias_allowed no)
     (uvia_min_size 0.2)
@@
     (solder_mask_min_width 0.25)
     (aux_axis_origin 0 0)
-    (visible_elements 7FFFF7FF)
+    (visible_elements 7FFFFFFF)
     (pcbplotparams
       (layerselection 0x010fc_ffffffff)
@@
   (net_class Default "This is the default net class."
     (clearance 0.2)
-    (trace_width 0.25)
-    (via_dia 0.8)
-    (via_drill 0.4)
-    (uvia_dia 0.3)
-    (uvia_drill 0.1)
-    (add_net +3V3)
-    (add_net +5V)
+    (trace_width 0.2)
+    (via_dia 0.6)
+    (via_drill 0.3)
+    (uvia_dia 0.6)
+    (uvia_drill 0.3)
     (add_net /A2)
     (add_net /Col0)
@@
     (add_net /SCL)
     (add_net /SDA)
-    (add_net GND)
     (add_net "Net-(CON1-Pad1)")
     (add_net "Net-(CON1-Pad2)")
@@
     (add_net "Net-(U3-Pad9)")
   )
-  (net_class Test ""
+  (net_class Power ""
     (clearance 0.2)
-    (trace_width 0.38)
-    (via_dia 0.8)
-    (via_drill 0.4)
-    (uvia_dia 0.3)
-    (uvia_drill 0.1)
+    (trace_width 0.7)
+    (via_dia 1)
+    (via_drill 0.5)
+    (uvia_dia 1)
+    (uvia_drill 0.5)
+    (add_net +3V3)
+    (add_net +5V)
+    (add_net GND)
   )
   (module digikey-footprints:Switch_Slide_11.6x4mm_SJ-3523-SMT (layer F.Cu)
@@
     (descr "D, DO-35_SOD27 series, Axial, Vertical, pin pitch=2.54mm, , length*diameter=4*2mm^2, , http://www.diodes.com/_files/packages/DO-35.pdf")
     (tags "D DO-35_SOD27 series Axial Vertical pin pitch 2.54mm  length 4mm diameter 2mm")
-    (fp_text reference D2 (at 1.27 -2.266371) (layer F.SilkS)
-      (effects (font (size 1 1) (thickness 0.15)))
-    )
+    (fp_text reference D2 (at 5.375 -0.1125) (layer F.SilkS)
+      (effects (font (size 1 1) (thickness 0.15)))
+    )

Commit message: Wire up the matrix to the io expander
Routing:
- net /Row0: track 0.00 -> 282.9 mm, vias 0 -> 1
- net /Row1: track 0.00 -> 276.0 mm, vias 0 -> 1
- net /ColD: track 0.00 -> 194.4 mm
- net /Col0: track 0.00 -> 172.8 mm
- net /ColC: track 0.00 -> 165.4 mm
- net /Col1: track 0.00 -> 159.4 mm
- net /ColB: track 0.00 -> 147.8 mm
- net /ColA: track 0.00 -> 129.3 mm
- net /Col2: track 0.00 -> 124.4 mm
- net /Col3: track 0.00 -> 121.3 mm
- net /Col4: track 0.00 -> 102.4 mm
- net /Col9: track 0.00 -> 96.5 mm
- net /Col8: track 0.00 -> 87.6 mm
- net /Col5: track 0.00 -> 83.6 mm
- net /Col7: track 0.00 -> 62.6 mm
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Other:
- net class Default: trace_width 0.2 -> 0.4; via_dia 0.6 -> 1; via_drill 0.3 -> 0.5
- net class Power: trace_width 0.7 -> 1

Commit message: Clean up the labels on the diodes a bit
Routing:
- net /ColA: track 129.3 -> 127.1 mm
- net /Col9: track 96.5 -> 94.3 mm
- net /Col8: track 87.6 -> 86.2 mm
- net /ColB: track 147.8 -> 146.9 mm

Commit message: Continue routing
Parts:
- removed J21: Control_7, Connectors_JST:JST_PH_S3B-PH-K_03x2.00mm_Angled
- removed R8: 10K, Resistors_THT:R_Axial_DIN0207_L6.3mm_D2.5mm_P7.62mm_Horizontal
- moved J23 0.20 mm to (278.0, 70.0)
- moved J10 0.15 mm to (90.2, 70.0)
- moved J13 0.15 mm to (153.7, 70.0)
- moved J18 0.15 mm to (215.9, 70.0)
Routing:
- net +3V3: track 0.00 -> 346.4 mm
- net GND: track 0.00 -> 311.5 mm, vias 0 -> 2
- net Net-(J4-Pad3): track 0.00 -> 52.1 mm
- net Net-(J4-Pad2): track 0.00 -> 52.1 mm
- net Net-(J4-Pad1): track 0.00 -> 52.1 mm
- net Net-(J3-Pad1): track 0.00 -> 39.6 mm
- net Net-(CON1-Pad1): track 0.00 -> 32.3 mm, vias 0 -> 2
- net Net-(J3-Pad2): track 0.00 -> 31.2 mm
- net Net-(J3-Pad3): track 0.00 -> 27.8 mm
- net Net-(CON1-Pad3): track 0.00 -> 26.7 mm
- net /POT1: track 0.00 -> 19.1 mm, vias 0 -> 2
- net /POT3: track 0.00 -> 18.8 mm, vias 0 -> 2
- net /POT0: track 0.00 -> 18.7 mm, vias 0 -> 2
- net /POT2: track 0.00 -> 18.5 mm, vias 0 -> 2
- net Net-(J10-Pad1): track 0.00 -> 16.6 mm
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Other:
- net class Small added: clearance 0.1, trace_width 0.2, via_dia 0.6, via_drill 0.3

Commit message: Finish connecting all pcb components
Connections:
- U1 pad 12: /POT3 -> /POT0
- U1 pad 13: /POT0 -> /POT1
- U1 pad 14: /POT1 -> /POT2
- U1 pad 15: /POT2 -> /POT3
- U1 pad 2: /POT6 -> /POT5
- U1 pad 4: /POT7 -> /POT6
- U1 pad 5: /POT5 -> /POT7
Routing:
- net +5V: track 9.37 -> 354.0 mm, vias 0 -> 1
- net GND: track 311.5 -> 585.7 mm, vias 2 -> 5
- net /SCL: track 0.00 -> 244.4 mm, vias 0 -> 1
- net /POT5: track 5.16 -> 247.9 mm
- net +3V3: track 346.4 -> 586.8 mm, vias 0 -> 3
- net /SDA: track 0.00 -> 237.7 mm, vias 0 -> 1
- net /POT6: track 6.79 -> 240.9 mm, vias 0 -> 1
- net /POT4: track 5.16 -> 230.7 mm, vias 0 -> 2
- net /A2: track 0.00 -> 170.6 mm, vias 0 -> 1
- net /POT3: track 18.8 -> 172.7 mm, vias 2 -> 1
- net /POT2: track 18.5 -> 107.0 mm, vias 2 -> 1
- net /D2: track 0.00 -> 83.5 mm, vias 0 -> 1
- net /D3: track 0.00 -> 82.5 mm, vias 0 -> 1
- net /D4: track 0.00 -> 81.1 mm, vias 0 -> 1
- net Net-(J12-Pad1): track 0.00 -> 72.5 mm, vias 0 -> 1
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
Commit message: Move audio plug down to leave room for 2U keycap
Parts:
- moved CON1 71.7 mm to (333.0, 140.2)
- moved CON2 57.0 mm to (330.0, 120.5), turned to 270 degrees
- moved U3 8.00 mm to (315.9, 90.0)
- moved J12 2.01 mm to (332.0, 55.9)
Routing:
- net Net-(CON1-Pad3): track 26.7 -> 49.2 mm
- net /SCL: track 244.4 -> 230.1 mm
- net /SDA: track 237.7 -> 223.3 mm
- net /A2: track 170.6 -> 158.7 mm
- net Net-(CON1-Pad1): track 32.3 -> 21.6 mm, vias 2 -> 0
- net +3V3: track 586.8 -> 576.3 mm
- net Net-(J12-Pad1): track 72.5 -> 80.8 mm, vias 1 -> 0
- net +5V: track 354.0 -> 349.6 mm, vias 1 -> 0
- net Net-(CON1-Pad2): track 12.5 -> 8.89 mm, vias 2 -> 0
- net /D2: track 83.5 -> 86.8 mm
- net /D8: track 33.6 -> 30.3 mm, vias 2 -> 1
- net Net-(J16-Pad3): track 9.78 -> 8.02 mm, vias 1 -> 0
- net /D3: track 82.5 -> 84.1 mm
- net Net-(J22-Pad3): track 9.36 -> 7.88 mm, vias 1 -> 0
- net Net-(J11-Pad3): track 9.47 -> 8.01 mm, vias 1 -> 0
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
Commit message: Change control and LED connectors and begin wiring
Parts:
- removed J18: LED_1_O, Connectors_JST:JST_PH_S3B-PH-K_03x2.00mm_Angled
- removed J19: LED_X_I, Pin_Headers:Pin_Header_Straight_1x03_Pitch2.54mm
- removed J20: Control_3, Connectors_JST:JST_PH_S3B-PH-K_03x2.00mm_Angled
- removed J22: LED_1_I, Connectors_JST:JST_PH_S3B-PH-K_03x2.00mm_Angled
- removed J23: LED_0_O, Connectors_JST:JST_PH_S3B-PH-K_03x2.00mm_Angled
- removed J24, J25: 10118193-0001LF, digikey-footprints:USB_Micro_B_Female_10118193-0001LF
- J1: value Control_0 -> 10118193-0001LF; footprint Connectors_JST:JST_PH_S3B-PH-K_03x2.00mm_Angled -> digikey-footprints:USB_Micro_B_Female_10118193-0001LF
- J10: value LED_3_O -> Control_LED_5_O; footprint Connectors_JST:JST_PH_S3B-PH-K_03x2.00mm_Angled -> Pin_Headers:Pin_Header_Angled_2x03_Pitch2.54mm
- J11, J16: footprint Connectors_JST:JST_PH_S3B-PH-K_03x2.00mm_Angled -> Pin_Headers:Pin_Header_Angled_1x03_Pitch2.54mm
- J12: value LED_0_I -> LED_X_O; footprint Connectors_JST:JST_PH_S3B-PH-K_03x2.00mm_Angled -> Pin_Headers:Pin_Header_Angled_1x03_Pitch2.54mm
- J13: value LED_2_O -> LED_X_I; footprint Connectors_JST:JST_PH_S3B-PH-K_03x2.00mm_Angled -> Pin_Headers:Pin_Header_Angled_1x03_Pitch2.54mm
- J14: value Control_2 -> Control_LED_1_O; footprint Connectors_JST:JST_PH_S3B-PH-K_03x2.00mm_Angled -> Pin_Headers:Pin_Header_Angled_2x03_Pitch2.54mm
- J15: value Control_6 -> Control_LED_4_O; footprint Connectors_JST:JST_PH_S3B-PH-K_03x2.00mm_Angled -> Pin_Headers:Pin_Header_Angled_2x03_Pitch2.54mm
- J17: value LED_X_O -> LED_5_I; footprint Pin_Headers:Pin_Header_Straight_1x03_Pitch2.54mm -> Pin_Headers:Pin_Header_Angled_1x03_Pitch2.54mm
- J2: value Control_4 -> Control_LED_0_O; footprint Connectors_JST:JST_PH_S3B-PH-K_03x2.00mm_Angled -> Pin_Headers:Pin_Header_Angled_2x03_Pitch2.54mm
- J3: value LED_4_O -> Control_LED_3_O; footprint Connectors_JST:JST_PH_S3B-PH-K_03x2.00mm_Angled -> Pin_Headers:Pin_Header_Angled_2x03_Pitch2.54mm
- J4: value LED_5_0 -> Control_LED_6_O; footprint Connectors_JST:JST_PH_S3B-PH-K_03x2.00mm_Angled -> Pin_Headers:Pin_Header_Angled_2x03_Pitch2.54mm
- J5: value LED_5_I -> 10118193-0001LF; footprint Connectors_JST:JST_PH_S3B-PH-K_03x2.00mm_Angled -> digikey-footprints:USB_Micro_B_Female_10118193-0001LF
- J6: value LED_4_I -> LED_1_I; footprint Connectors_JST:JST_PH_S3B-PH-K_03x2.00mm_Angled -> Pin_Headers:Pin_Header_Angled_1x03_Pitch2.54mm
- J7: value Control_1 -> LED_4_I; footprint Connectors_JST:JST_PH_S3B-PH-K_03x2.00mm_Angled -> Pin_Headers:Pin_Header_Angled_1x03_Pitch2.54mm
- J8: value Control_5 -> LED_0_I; footprint Connectors_JST:JST_PH_S3B-PH-K_03x2.00mm_Angled -> Pin_Headers:Pin_Header_Angled_1x03_Pitch2.54mm
- J9: value LED_6_I -> Control_LED_2_O; footprint Connectors_JST:JST_PH_S3B-PH-K_03x2.00mm_Angled -> Pin_Headers:Pin_Header_Angled_2x03_Pitch2.54mm
- moved J8 303.6 mm to (315.5, 62.0), turned to 0 degrees
- moved J1 296.1 mm to (-24.5, 36.0), turned to 180 degrees
- moved J2 275.7 mm to (298.5, 67.0), turned to 180 degrees
- moved J17 248.8 mm to (25.5, 108.5), turned to 90 degrees
- moved R6 221.9 mm to (240.5, 68.0)
- moved R4 173.8 mm to (178.0, 68.0), turned to 90 degrees
- moved J6 169.2 mm to (253.0, 62.0), turned to 0 degrees
- moved R3 153.0 mm to (53.0, 84.0)
- moved J7 142.8 mm to (65.5, 61.5), turned to 0 degrees
- moved J9 142.5 mm to (174.0, 67.0)
- moved D12 141.3 mm to (272.5, 81.8)
- moved D10 138.8 mm to (152.4, 109.5), turned to 0 degrees
- moved R5 126.3 mm to (31.5, 123.0), turned to 180 degrees
- moved J13 116.1 mm to (269.5, 78.5), turned to 180 degrees
- moved R2 96.6 mm to (115.5, 68.0)
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Connections:
- D10 pad 1: Net-(D10-Pad1) -> /Col5
- D10 pad 2: +5V -> Net-(D10-Pad2)
- D12 pad 1: /Col5 -> Net-(D12-Pad1)
- D12 pad 2: Net-(D12-Pad2) -> +5V
- J1 pad 1: +3V3 -> Net-(J1-Pad1)
- J1 pad 2: /POT0 -> Net-(J1-Pad2)
- J1 pad 3: GND -> Net-(J1-Pad3)
- J10 pad 2: Net-(J10-Pad2) -> +3V3
- J12 pad 1: Net-(J12-Pad1) -> (no net)
- J12 pad 2: +5V -> Net-(J12-Pad2)
- J13 pad 1: Net-(J11-Pad1) -> Net-(D12-Pad1)
- J13 pad 2: Net-(J11-Pad2) -> /D8
- J13 pad 3: Net-(J11-Pad3) -> GND
- J14 pad 1: +3V3 -> Net-(J14-Pad1)
- J14 pad 2: /POT2 -> +3V3
- J14 pad 3: GND -> Net-(J14-Pad3)
- J15 pad 1: +3V3 -> Net-(J15-Pad1)
- J15 pad 2: /POT6 -> +3V3
- J15 pad 3: GND -> Net-(J15-Pad3)
- J16 pad 1: Net-(J16-Pad1) -> Net-(J14-Pad5)
- J16 pad 2: Net-(J16-Pad2) -> Net-(J14-Pad3)
- J16 pad 3: Net-(J16-Pad3) -> Net-(J14-Pad1)
- J17 pad 1: Net-(J12-Pad1) -> Net-(J15-Pad5)
- J17 pad 2: Net-(J17-Pad2) -> Net-(J15-Pad3)
- J17 pad 3: Net-(J12-Pad3) -> Net-(J15-Pad1)
- J2 pad 1: +3V3 -> Net-(J2-Pad1)
- J2 pad 2: /POT4 -> +3V3
- J2 pad 3: GND -> Net-(J2-Pad3)
- J3 pad 2: Net-(J3-Pad2) -> +3V3
- J4 pad 1: Net-(J4-Pad1) -> Net-(J10-Pad1)
- J4 pad 2: Net-(J4-Pad2) -> +3V3
- J4 pad 3: Net-(J4-Pad3) -> Net-(J10-Pad3)
- J5 pad 1: Net-(J3-Pad1) -> Net-(J1-Pad1)
- J5 pad 2: Net-(J3-Pad2) -> Net-(J1-Pad2)
- J5 pad 3: Net-(J3-Pad3) -> Net-(J1-Pad3)
- J6 pad 1: Net-(J10-Pad1) -> Net-(J2-Pad5)
- J6 pad 2: Net-(J10-Pad2) -> Net-(J2-Pad3)
- J6 pad 3: Net-(J10-Pad3) -> Net-(J2-Pad1)
- J7 pad 1: +3V3 -> Net-(J3-Pad5)
- J7 pad 2: /POT1 -> Net-(J3-Pad3)
- J7 pad 3: GND -> Net-(J3-Pad1)
- J8 pad 1: +3V3 -> Net-(J12-Pad3)
- J8 pad 2: /POT5 -> Net-(J12-Pad2)
- J8 pad 3: GND -> +5V
- J9 pad 1: Net-(J4-Pad1) -> Net-(J11-Pad3)
- J9 pad 2: Net-(J4-Pad2) -> +3V3
- J9 pad 3: Net-(J4-Pad3) -> Net-(J11-Pad2)
- R2 pad 1: /POT4 -> /POT3
- R3 pad 1: /POT1 -> /POT6
- R4 pad 1: /POT5 -> /POT2
- R5 pad 1: /POT2 -> /POT5
- R6 pad 1: /POT6 -> /POT1
- R7 pad 1: /POT3 -> /POT4
- S10 pad 2: Net-(D11-Pad2) -> Net-(D10-Pad2)
- S11 pad 2: Net-(D12-Pad2) -> Net-(D11-Pad2)
- U1 pad 5: /POT7 -> (no net)
- U2 pad 11: Net-(U2-Pad11) -> (no net)
- U2 pad 14: Net-(U2-Pad14) -> (no net)
- U2 pad 19: Net-(U2-Pad19) -> (no net)
- U2 pad 20: Net-(U2-Pad20) -> (no net)
- U3 pad 11: Net-(U3-Pad11) -> (no net)
- U3 pad 12: Net-(U3-Pad12) -> (no net)
- U3 pad 13: Net-(U3-Pad13) -> (no net)
- U3 pad 14: Net-(U3-Pad14) -> (no net)
- U3 pad 15: Net-(U3-Pad15) -> (no net)
- U3 pad 17: Net-(U3-Pad17) -> (no net)
- U3 pad 18: Net-(U3-Pad18) -> (no net)
- U3 pad 19: Net-(U3-Pad19) -> (no net)
- U3 pad 2: Net-(U3-Pad2) -> (no net)
- U3 pad 20: Net-(U3-Pad20) -> (no net)
- U3 pad 21: Net-(U3-Pad21) -> (no net)
- U3 pad 22: Net-(U3-Pad22) -> (no net)
- U3 pad 24: Net-(U3-Pad24) -> (no net)
- U3 pad 27: Net-(U3-Pad27) -> (no net)
- U3 pad 28: Net-(U3-Pad28) -> (no net)
- U3 pad 29: Net-(U3-Pad29) -> (no net)
- U3 pad 3: Net-(U3-Pad3) -> (no net)
- U3 pad 30: Net-(U3-Pad30) -> (no net)
- U3 pad 31: Net-(U3-Pad31) -> (no net)
- U3 pad 32: Net-(U3-Pad32) -> (no net)
- U3 pad 33: Net-(U3-Pad33) -> (no net)
- U3 pad 34: Net-(U3-Pad34) -> (no net)
- U3 pad 35: Net-(U3-Pad35) -> (no net)
- U3 pad 36: Net-(U3-Pad36) -> (no net)
- U3 pad 37: Net-(U3-Pad37) -> (no net)
- U3 pad 38: Net-(U3-Pad38) -> (no net)
- U3 pad 39: Net-(U3-Pad39) -> (no net)
- U3 pad 40: Net-(U3-Pad40) -> (no net)
- U3 pad 41: Net-(U3-Pad41) -> (no net)
- U3 pad 42: Net-(U3-Pad42) -> (no net)
- U3 pad 43: Net-(U3-Pad43) -> (no net)
- U3 pad 44: Net-(U3-Pad44) -> (no net)
- U3 pad 45: Net-(U3-Pad45) -> (no net)
- U3 pad 46: Net-(U3-Pad46) -> (no net)
- U3 pad 47: Net-(U3-Pad47) -> (no net)
- U3 pad 48: Net-(U3-Pad48) -> (no net)
- U3 pad 49: Net-(U3-Pad49) -> (no net)
- U3 pad 50: Net-(U3-Pad50) -> (no net)
- U3 pad 51: Net-(U3-Pad51) -> (no net)
- U3 pad 7: /D5 -> (no net)
- U3 pad 8: Net-(U3-Pad8) -> (no net)
- U3 pad 9: Net-(U3-Pad9) -> (no net)
Routing:
- net GND: track 584.8 -> 111.9 mm, vias 5 -> 2
- net +5V: track 349.6 -> 0.00 mm
- net +3V3: track 576.3 -> 245.4 mm, vias 3 -> 4
- net /POT5: track 247.5 -> 0.00 mm
- net /POT6: track 240.9 -> 0.00 mm, vias 1 -> 0
- net /POT4: track 230.7 -> 0.00 mm, vias 2 -> 0
- net /POT3: track 172.7 -> 0.00 mm, vias 1 -> 0
- net /POT2: track 107.0 -> 0.00 mm, vias 1 -> 0
- net Net-(J12-Pad1): track 80.8 -> 0.00 mm
- net Net-(J2-Pad1): track 0.00 -> 78.2 mm
- net Net-(J14-Pad3): track 0.00 -> 69.8 mm
- net Net-(J2-Pad3): track 0.00 -> 69.7 mm
- net Net-(J12-Pad3): track 68.9 -> 0.00 mm
- net Net-(J4-Pad3): track 52.1 -> 0.00 mm
- net Net-(J4-Pad2): track 52.1 -> 0.00 mm
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