File: teensynth.kicad_pcb (KiCad board)
At the start: 2 copper layers, 80 parts, among them CON1 SJ-3523-SMT-TR, CON2 SJ-3523-SMT-TR, J1 10118193-0001LF, J10 Control_LED_5_O, J11 LED_3_I, J12 LED_X_O, J13 LED_X_I, J14 Control_LED_1_O, J15 Control_LED_4_O, J16 LED_2_I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

Commit message: Begin improving control and led connections
Parts:
- moved J13 5.41 mm to (266.5, 83.0)
- moved J12 2.26 mm to (242.2, 78.2)
Routing:
- net GND: track 111.9 -> 424.7 mm
- net +3V3: track 245.4 -> 465.9 mm, vias 4 -> 3
- net /POT2: track 0.00 -> 73.0 mm, vias 0 -> 1
- net Net-(J11-Pad1): track 0.00 -> 47.1 mm
- net Net-(J11-Pad2): track 0.00 -> 47.1 mm
- net Net-(J14-Pad1): track 0.00 -> 47.1 mm
- net Net-(J11-Pad3): track 0.00 -> 47.1 mm
- net Net-(J2-Pad1): track 78.2 -> 46.6 mm
- net Net-(J2-Pad3): track 69.7 -> 46.6 mm
- net Net-(J14-Pad3): track 69.8 -> 47.1 mm
- net Net-(J14-Pad5): track 48.9 -> 47.1 mm
- net /POT1: track 47.3 -> 46.1 mm
- net Net-(J2-Pad5): track 48.4 -> 47.3 mm
- net /POT0: track 104.8 -> 104.0 mm

Commit message: Finish wiring nearly all new connectors
Parts:
- moved J5 230.9 mm to (239.5, 30.5), turned to 90 degrees
- moved J1 55.4 mm to (18.0, 71.5), turned to 270 degrees
- moved D12 48.8 mm to (281.5, 33.8)
- moved J12 48.8 mm to (251.2, 30.2)
- moved J13 48.8 mm to (275.5, 35.0)
- moved R3 0.50 mm to (53.0, 83.5)
Routing:
- net GND: track 424.7 -> 757.0 mm, vias 2 -> 1
- net /POT5: track 0.00 -> 255.2 mm, vias 0 -> 1
- net /POT6: track 0.00 -> 217.2 mm, vias 0 -> 1
- net /POT4: track 0.00 -> 210.1 mm, vias 0 -> 1
- net /POT3: track 0.00 -> 140.6 mm, vias 0 -> 1
- net +3V3: track 465.9 -> 556.3 mm
- net Net-(J10-Pad5): track 0.00 -> 65.3 mm
- net Net-(J15-Pad5): track 0.00 -> 63.2 mm
- net Net-(J15-Pad3): track 0.00 -> 58.4 mm
- net Net-(J10-Pad3): track 0.00 -> 56.2 mm
- net Net-(J15-Pad1): track 0.00 -> 52.8 mm
- net Net-(J10-Pad1): track 0.00 -> 51.7 mm
- net Net-(J3-Pad1): track 0.00 -> 46.9 mm
- net Net-(J3-Pad3): track 0.00 -> 46.9 mm
- net Net-(J3-Pad5): track 0.00 -> 46.9 mm
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
Commit message: Wire usb port and LED x
Parts:
- moved J5 219.7 mm to (21.9, 61.5)
- moved J12 53.9 mm to (262.5, 83.0), turned to 180 degrees
- moved D12 49.3 mm to (282.5, 83.0)
- moved J13 48.1 mm to (278.5, 83.0)
Routing:
- net Net-(J12-Pad3): track 0.00 -> 59.6 mm
- net Net-(J12-Pad2): track 0.00 -> 59.6 mm
- net /D8: track 0.00 -> 45.4 mm, vias 0 -> 1
- net GND: track 757.0 -> 796.1 mm, vias 1 -> 2
- net +5V: track 0.00 -> 37.1 mm
- net Net-(J1-Pad3): track 0.00 -> 36.7 mm
- net Net-(J1-Pad4): track 0.00 -> 33.9 mm, vias 0 -> 2
- net Net-(J1-Pad2): track 0.00 -> 16.0 mm, vias 0 -> 2
- net Net-(J1-Pad1): track 0.00 -> 11.6 mm
- net Net-(D12-Pad1): track 0.00 -> 4.02 mm

Commit message: Finish wiring up PCB
Parts:
- J4: value Control_LED_6_O -> Control_LED_6_I
- J5: footprint digikey-footprints:USB_Micro_B_Female_10118193-0001LF -> Pin_Headers:Pin_Header_Straight_1x05_Pitch2.54mm
- moved J1 317.0 mm to (335.0, 74.2), turned to 90 degrees
- moved J5 311.8 mm to (333.0, 83.0), turned to 0 degrees
- moved CON1 8.01 mm to (333.4, 132.2)
- moved CON2 6.20 mm to (330.0, 114.3)
Connections:
- J1 pad 1: Net-(J1-Pad1) -> +5V
- J1 pad 5: GND -> Net-(J1-Pad5)
- J12 pad 1: (no net) -> Net-(J12-Pad1)
- J5 pad 1: Net-(J1-Pad1) -> +5V
- J5 pad 5: GND -> Net-(J1-Pad5)
- U1 pad 5: (no net) -> Net-(U1-Pad5)
- U2 pad 11: (no net) -> Net-(U2-Pad11)
- U2 pad 14: (no net) -> Net-(U2-Pad14)
- U2 pad 19: (no net) -> Net-(U2-Pad19)
- U2 pad 20: (no net) -> Net-(U2-Pad20)
- U3 pad 11: (no net) -> Net-(U3-Pad11)
- U3 pad 12: (no net) -> Net-(U3-Pad12)
- U3 pad 13: (no net) -> Net-(U3-Pad13)
- U3 pad 14: (no net) -> Net-(U3-Pad14)
- U3 pad 15: (no net) -> Net-(U3-Pad15)
- U3 pad 17: (no net) -> Net-(U3-Pad17)
- U3 pad 18: (no net) -> Net-(U3-Pad18)
- U3 pad 19: (no net) -> Net-(U3-Pad19)
- U3 pad 2: (no net) -> Net-(U3-Pad2)
- U3 pad 20: (no net) -> Net-(U3-Pad20)
- U3 pad 21: (no net) -> Net-(U3-Pad21)
- U3 pad 22: (no net) -> Net-(U3-Pad22)
- U3 pad 24: (no net) -> Net-(U3-Pad24)
- U3 pad 27: (no net) -> Net-(U3-Pad27)
- U3 pad 28: (no net) -> Net-(U3-Pad28)
- U3 pad 29: (no net) -> Net-(U3-Pad29)
- U3 pad 3: (no net) -> Net-(U3-Pad3)
- U3 pad 30: (no net) -> Net-(U3-Pad30)
- U3 pad 31: (no net) -> Net-(U3-Pad31)
- U3 pad 32: (no net) -> Net-(U3-Pad32)
- U3 pad 33: (no net) -> Net-(U3-Pad33)
- U3 pad 34: (no net) -> Net-(U3-Pad34)
- U3 pad 35: (no net) -> Net-(U3-Pad35)
- U3 pad 36: (no net) -> Net-(U3-Pad36)
- U3 pad 37: (no net) -> Net-(U3-Pad37)
- U3 pad 38: (no net) -> Net-(U3-Pad38)
- U3 pad 39: (no net) -> Net-(U3-Pad39)
- U3 pad 40: (no net) -> Net-(U3-Pad40)
- U3 pad 41: (no net) -> Net-(U3-Pad41)
- U3 pad 42: (no net) -> Net-(U3-Pad42)
- U3 pad 43: (no net) -> Net-(U3-Pad43)
- U3 pad 44: (no net) -> Net-(U3-Pad44)
- U3 pad 45: (no net) -> Net-(U3-Pad45)
- U3 pad 46: (no net) -> Net-(U3-Pad46)
- U3 pad 47: (no net) -> Net-(U3-Pad47)
- U3 pad 48: (no net) -> Net-(U3-Pad48)
- U3 pad 49: (no net) -> Net-(U3-Pad49)
- U3 pad 50: (no net) -> Net-(U3-Pad50)
- U3 pad 51: (no net) -> Net-(U3-Pad51)
- U3 pad 7: (no net) -> /D5
- U3 pad 8: (no net) -> Net-(U3-Pad8)
- U3 pad 9: (no net) -> Net-(U3-Pad9)
Routing:
- net +5V: track 37.1 -> 76.5 mm
- net Net-(J1-Pad5): track 0.00 -> 24.2 mm
- net Net-(J1-Pad3): track 36.7 -> 16.6 mm
- net Net-(J1-Pad4): track 33.9 -> 20.4 mm, vias 2 -> 0
- net Net-(J1-Pad1): track 11.6 -> 0.00 mm
- net GND: track 796.1 -> 788.6 mm, vias 2 -> 0
- net Net-(J1-Pad2): track 16.0 -> 12.8 mm, vias 2 -> 0
- net Net-(CON1-Pad2): track 8.89 -> 6.93 mm
- net Net-(CON1-Pad3): track 49.2 -> 51.0 mm
- net Net-(CON1-Pad1): track 21.6 -> 20.1 mm

Commit message: Minor PCB improvements
Parts:
- J5: value 10118193-0001LF -> USB
Routing:
- net /POT5: track 255.2 -> 250.3 mm
- net +3V3: track 556.3 -> 552.8 mm
- net /A2: track 177.0 -> 173.8 mm
- net /POT0: track 104.0 -> 104.8 mm
